Commit message: Integrate GPU terrain navigation baseline
Add modular Isaac simulation launchers, dynamic map clearing, FSGP-BGK SE2 terrain integration, planner updates, tests, and experiment documentation.

File: src/simulator/fake_ugv/hunter_se/hunter_se_gazebo/xacro/hunter_se_gazebo.xacro (robot description, xacro)
@@ -8,4 +8,5 @@
   <xacro:arg name="enable_livox" default="true" />
   <xacro:arg name="enable_d455" default="true" />
+  <xacro:arg name="enable_suspension" default="false" />
   <xacro:include filename="$(find hunter_se_gazebo)/xacro/hunter_se.gazebo" />
   <xacro:include filename="$(find ros2_livox_simulation)/urdf/mid360.xacro" />
@@ -26,4 +27,5 @@
   <xacro:property name="rear_wheel_radius" value="0.13495" />
   <xacro:property name="rear_wheel_width" value="0.1540" />
+  <xacro:property name="enable_suspension_value" value="$(arg enable_suspension)" />
   <xacro:property name="locked_planar_drive_mode" value="${drive_mode_value == 'planar'}" />
   <xacro:property name="planar_visual_drive_mode" value="${drive_mode_value == 'planar_visual'}" />
@@ -72,4 +74,31 @@
     </collision>
   </link>
+  <link name="fr_susp_left_link">
+    <inertial>
+      <origin xyz="0 0 0" rpy="0 0 0" />
+      <mass value="0.20" />
+      <inertia ixx="0.001" ixy="0" ixz="0" iyy="0.001" iyz="0" izz="0.001" />
+    </inertial>
+    <visual>
+      <geometry><box size="0.001 0.001 0.001" /></geometry>
+    </visual>
+  </link>
+  <xacro:if value="${enable_suspension_value}">
+    <joint name="fr_susp_left_joint" type="prismatic">
+      <origin xyz="0.34058 0.24619 -0.1535" rpy="0 0 0" />
+      <parent link="base_link" />
+      <child link="fr_susp_left_link" />
+      <axis xyz="0 0 1" />
+      <limit lower="-0.040" upper="0.040" effort="1200" velocity="0.8" />
+      <dynamics damping="45.0" friction="1.0" />
+    </joint>
+  </xacro:if>
+  <xacro:unless value="${enable_suspension_value}">
+    <joint name="fr_susp_left_joint" type="fixed">
+      <origin xyz="0.34058 0.24619 -0.1535" rpy="0 0 0" />
+      <parent link="base_link" />
+      <child link="fr_susp_left_link" />
+    </joint>
+  </xacro:unless>
   <link
     name="fr_steer_left_link">
@@ -114,8 +143,8 @@
     type="revolute">
     <origin
-      xyz="0.34058 0.24619 -0.1535"
+      xyz="0 0 0"
       rpy="0 0 0" />
     <parent
-      link="base_link" />
+      link="fr_susp_left_link" />
     <child
       link="fr_steer_left_link" />
@@ -180,6 +209,33 @@
     <axis
       xyz="0 0 -1" />
-    <dynamics damping="0.35" friction="0.08" />
+    <dynamics damping="0.02" friction="0.01" />
   </joint>
+  <link name="fr_susp_right_link">
+    <inertial>
+      <origin xyz="0 0 0" rpy="0 0 0" />
+      <mass value="0.20" />
+      <inertia ixx="0.001" ixy="0" ixz="0" iyy="0.001" iyz="0" izz="0.001" />
+    </inertial>
+    <visual>
+      <geometry><box size="0.001 0.001 0.001" /></geometry>
+    </visual>
+  </link>
+  <xacro:if value="${enable_suspension_value}">
+    <joint name="fr_susp_right_joint" type="prismatic">
+      <origin xyz="0.34219 -0.24619 -0.1535" rpy="0 0 0" />
+      <parent link="base_link" />
+      <child link="fr_susp_right_link" />
+      <axis xyz="0 0 1" />
+      <limit lower="-0.040" upper="0.040" effort="1200" velocity="0.8" />
+      <dynamics damping="45.0" friction="1.0" />
+    </joint>
+  </xacro:if>
+  <xacro:unless value="${enable_suspension_value}">
+    <joint name="fr_susp_right_joint" type="fixed">
+      <origin xyz="0.34219 -0.24619 -0.1535" rpy="0 0 0" />
+      <parent link="base_link" />
+      <child link="fr_susp_right_link" />
+    </joint>
+  </xacro:unless>
   <link
     name="fr_steer_right_link">
@@ -224,8 +280,8 @@
     type="revolute">
     <origin
-      xyz="0.34219 -0.24619 -0.1535"
+      xyz="0 0 0"
       rpy="0 0 0" />
     <parent
-      link="base_link" />
+      link="fr_susp_right_link" />
     <child
       link="fr_steer_right_link" />
@@ -290,6 +346,33 @@
     <axis
       xyz="0 0 1" />
-    <dynamics damping="0.35" friction="0.08" />
+    <dynamics damping="0.02" friction="0.01" />
   </joint>
+  <link name="re_susp_left_link">
+    <inertial>
+      <origin xyz="0 0 0" rpy="0 0 0" />
+      <mass value="0.20" />
+      <inertia ixx="0.001" ixy="0" ixz="0" iyy="0.001" iyz="0" izz="0.001" />
+    </inertial>
+    <visual>
+      <geometry><box size="0.001 0.001 0.001" /></geometry>
+    </visual>
+  </link>
+  <xacro:if value="${enable_suspension_value}">
+    <joint name="re_susp_left_joint" type="prismatic">
+      <origin xyz="-0.2078 0.252 -0.158" rpy="0 0 0" />
+      <parent link="base_link" />
+      <child link="re_susp_left_link" />
+      <axis xyz="0 0 1" />
+      <limit lower="-0.040" upper="0.040" effort="1200" velocity="0.8" />
+      <dynamics damping="45.0" friction="1.0" />
+    </joint>
+  </xacro:if>
+  <xacro:unless value="${enable_suspension_value}">
+    <joint name="re_susp_left_joint" type="fixed">
+      <origin xyz="-0.2078 0.252 -0.158" rpy="0 0 0" />
+      <parent link="base_link" />
+      <child link="re_susp_left_link" />
+    </joint>
+  </xacro:unless>
   <link
     name="re_left_link">
@@ -335,14 +418,41 @@
     type="continuous">
     <origin
-      xyz="-0.2078 0.252 -0.158"
+      xyz="0 0 0"
       rpy="1.5708 0 0" />
     <parent
-      link="base_link" />
+      link="re_susp_left_link" />
     <child
       link="re_left_link" />
     <axis
       xyz="0 0 -1" />
-    <dynamics damping="0.35" friction="0.08" />
+    <dynamics damping="0.02" friction="0.01" />
   </joint>
+  <link name="re_susp_right_link">
+    <inertial>
+      <origin xyz="0 0 0" rpy="0 0 0" />
+      <mass value="0.20" />
+      <inertia ixx="0.001" ixy="0" ixz="0" iyy="0.001" iyz="0" izz="0.001" />
+    </inertial>
+    <visual>
+      <geometry><box size="0.001 0.001 0.001" /></geometry>
+    </visual>
+  </link>
+  <xacro:if value="${enable_suspension_value}">
+    <joint name="re_susp_right_joint" type="prismatic">
+      <origin xyz="-0.2078 -0.252 -0.158" rpy="0 0 0" />
+      <parent link="base_link" />
+      <child link="re_susp_right_link" />
+      <axis xyz="0 0 1" />
+      <limit lower="-0.040" upper="0.040" effort="1200" velocity="0.8" />
+      <dynamics damping="45.0" friction="1.0" />
+    </joint>
+  </xacro:if>
+  <xacro:unless value="${enable_suspension_value}">
+    <joint name="re_susp_right_joint" type="fixed">
+      <origin xyz="-0.2078 -0.252 -0.158" rpy="0 0 0" />
+      <parent link="base_link" />
+      <child link="re_susp_right_link" />
+    </joint>
+  </xacro:unless>
   <link
     name="re_right_link">
@@ -388,13 +498,13 @@
     type="continuous">
     <origin
-      xyz="-0.2078 -0.252 -0.158"
+      xyz="0 0 0"
       rpy="-1.5708 0 0" />
     <parent
-      link="base_link" />
+      link="re_susp_right_link" />
     <child
       link="re_right_link" />
     <axis
       xyz="0 0 1" />
-    <dynamics damping="0.35" friction="0.08" />
+    <dynamics damping="0.02" friction="0.01" />
   </joint>
    <link name="steering_wheel_link">
